File: Houston Board v.1.0/Houston Board v1.1.brd (EAGLE design)
At the start: 86 x 86 mm, 69 parts, among them IC2 TP4056, IC5 TESEO-LIV3F, IC6 BGA_725L6_E6327, IC7 ST1S12GR, P2 53398-0610, T2 DMN3024LSD, U2 MP2307DN-LF-Z, U3 FT232RLSSOP, U4 MAX40200AUK+, U5 MAX40200AUK+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

Commit message: Add files via upload
Parts:
- 3V3, TX1: value Red -> (none)
- C12: value 10uf -> 10uF
- C2: value 0.1u -> 0.1uF
- C20: value 1onF -> 10nF
- R1: value 220R -> 220
- R14: value 1.5K -> 1.5k
- R2: value 120R -> 120
- R3, R4: value 1K -> 1k
- R5: value 100K -> 100k
- R6: value 6.8K -> 6.8k
- R7: value 26.1K -> 26.1k
- R8: value 10K -> 10k
- RX1: value Green -> (none)
