File: Houston Board v.1.0/Houston Board v1.1.sch (EAGLE design)
At the start: 71 parts, among them IC2 TP4056, IC5 TESEO-LIV3F, IC6 BGA_725L6_E6327, IC7 ST1S12GR, P2 53398-0610, T2 DMN3024LSD, U2 MP2307DN-LF-Z, U3 FT232RLSSOP, U4 MAX40200AUK+, U5 MAX40200AUK+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

Commit message: Correção de Erros
Parts:
- removed R17, R18: (no value), rcl:R-EU_R0805
- L2-7,5NH1: value 0603CS-7N5XGLU -> LQW18AS7N5J0ZD; device SamacSys_Parts:0603CS-7N5XGLU -> LQW18AS7N5J0ZD:LQW18AS7N5J0ZD
- R14: value (none) -> 1.5K
- R2: value (none) -> 120R
- U$3: value LTF5022T100M1R4-LC -> LTF5022T100M1R4; device mylbr:LTF5022T100M1R4-LC -> LTF5022T:LTF5022T100M1R4
Connections:
- removed net N$37: IC2.TEMP, R17.1, R18.2
- net 5V: no longer R17.2
- net GND: now also IC2.TEMP; no longer R18.1
- net NSS_BUS: now also U6.SCS/CMD
- net UART_RX_BUS: no longer U6.IO16
- net UART_TX_BUS: no longer U6.IO17
Other:
- note added: "Diodo DCDC"
- note added: "Diodo FTDI"
- note added: "Resistor de Programação : 1K - 780mA(Ibat)"
Changed lines of the file:
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@@
 <?xml version="1.0" encoding="utf-8"?>
 <!DOCTYPE eagle SYSTEM "eagle.dtd">
-<eagle version="9.6.1">
+<eagle version="9.5.2">
 <drawing>
 <settings>
@@
 <part name="U$2" library="DW01" deviceset="DW01" device=""/>
 <part name="GND19" library="supply1" library_urn="urn:adsk.eagle:library:371" deviceset="GND" device=""/>
-<part name="R14" library="rcl" library_urn="urn:adsk.eagle:library:334" deviceset="R-EU_" device="R0805" package3d_urn="urn:adsk.eagle:package:23553/2"/>
+<part name="R14" library="rcl" library_urn="urn:adsk.eagle:library:334" deviceset="R-EU_" device="R0805" package3d_urn="urn:adsk.eagle:package:23553/2" value="1.5K"/>
 <part name="GND20" library="supply1" library_urn="urn:adsk.eagle:library:371" deviceset="GND" device=""/>
 <part name="R15" library="rcl" library_urn="urn:adsk.eagle:library:334" deviceset="R-EU_" device="R0805" package3d_urn="urn:adsk.eagle:package:23553/2" value="1k"/>
@@
 <part name="CHRG1" library="led" library_urn="urn:adsk.eagle:library:259" deviceset="LED" device="CHIP-LED0805" package3d_urn="urn:adsk.eagle:package:15818/2"/>
 <part name="STD1" library="led" library_urn="urn:adsk.eagle:library:259" deviceset="LED" device="CHIP-LED0805" package3d_urn="urn:adsk.eagle:package:15818/2"/>
-<part name="R17" library="rcl" library_urn="urn:adsk.eagle:library:334" deviceset="R-EU_" device="R0805" package3d_urn="urn:adsk.eagle:package:23553/2"/>
-<part name="R18" library="rcl" library_urn="urn:adsk.eagle:library:334" deviceset="R-EU_" device="R0805" package3d_urn="urn:adsk.eagle:package:23553/2"/>
 <part name="GND21" library="supply1" library_urn="urn:adsk.eagle:library:371" deviceset="GND" device=""/>
 <part name="C12" library="rcl" library_urn="urn:adsk.eagle:library:334" deviceset="C-EU" device="C0805" package3d_urn="urn:adsk.eagle:package:23617/2" value="10uf"/>
@@
 <part name="C21" library="rcl" library_urn="urn:adsk.eagle:library:334" deviceset="C-EU" device="C1206" package3d_urn="urn:adsk.eagle:package:23618/2" value="56pF"/>
 <part name="L4-27NH1" library="SamacSys_Parts" deviceset="LQG15HS27NJ02D" device=""/>
-<part name="L2-7,5NH1" library="SamacSys_Parts" deviceset="0603CS-7N5XGLU" device=""/>
+<part name="L2-7,5NH1" library="LQW18AS7N5J0ZD" deviceset="LQW18AS7N5J0ZD" device=""/>
 <part name="IC7" library="SamacSys_Parts" deviceset="ST1S12GR" device=""/>
 <part name="C22" library="rcl" library_urn="urn:adsk.eagle:library:334" deviceset="C-EU" device="C1206" package3d_urn="urn:adsk.eagle:package:23618/2" value="56pF"/>
@@
 <part name="C23" library="rcl" library_urn="urn:adsk.eagle:library:334" deviceset="C-EU" device="C1206" package3d_urn="urn:adsk.eagle:package:23618/2" value="22uF"/>
 <part name="GND48" library="supply1" library_urn="urn:adsk.eagle:library:371" deviceset="GND" device=""/>
-<part name="U$3" library="mylbr" deviceset="LTF5022T" device="100M1R4-LC"/>
+<part name="U$3" library="LTF5022T" deviceset="LTF5022T" device="100M1R4"/>
 <part name="U6" library="ESP32-WROOM-32D" deviceset="ESP32-WROOM-32D" device=""/>
 <part name="COMM_CAN_TRANSCEIVER1" library="SN65HVD233D" deviceset="SN65HVD233D" device=""/>
@@
 <part name="S2" library="SparkFun-Switches" deviceset="MOMENTARY-SWITCH-SPST" device="-SMD-6.0X3.5MM"/>
 <part name="P2" library="con-molex-picoblade" deviceset="53398-0610" device=""/>
-<part name="R2" library="rcl" library_urn="urn:adsk.eagle:library:334" deviceset="R-EU_" device="R0805" package3d_urn="urn:adsk.eagle:package:23553/2"/>
+<part name="R2" library="rcl" library_urn="urn:adsk.eagle:library:334" deviceset="R-EU_" device="R0805" package3d_urn="urn:adsk.eagle:package:23553/2" value="120R"/>
 </parts>
 <sheets>
@@
 <wire x1="551.18" y1="-30.48" x2="551.18" y2="28.448" width="0.1524" layer="94"/>
 <text x="597.66" y="22.24" size="5.08" layer="94">ESP32-WROOM</text>
+<text x="449.58" y="30.48" size="1.778" layer="95">Resistor de Programação : 1K - 780mA(Ibat)</text>
+<text x="363.22" y="170.18" size="2.54" layer="94">Diodo DCDC</text>
+<text x="363.22" y="129.54" size="2.54" layer="94">Diodo FTDI</text>
 </plain>
 <instances>
@@
 <attribute name="VALUE" x="529.435" y="69.548" size="1.778" layer="96" rot="R90"/>
 </instance>
-<instance part="R17" gate="G$1" x="448.282" y="67.262" smashed="yes" rot="R90">
-<attribute name="NAME" x="446.7834" y="63.452" size="1.778" layer="95" rot="R90"/>
-<attribute name="VALUE" x="451.584" y="63.452" size="1.778" layer="96" rot="R90"/>
-</instance>
-<instance part="R18" gate="G$1" x="448.282" y="49.228" smashed="yes" rot="R90">
-<attribute name="NAME" x="446.7834" y="45.418" size="1.778" layer="95" rot="R90"/>
-<attribute name="VALUE" x="451.584" y="45.418" size="1.778" layer="96" rot="R90"/>
-</instance>
 <instance part="GND21" gate="1" x="448.282" y="37.036" smashed="yes">
 <attribute name="VALUE" x="445.742" y="34.496" size="1.778" layer="96"/>
@@
 <attribute name="VALUE" x="435.61" y="6.35" size="1.778" layer="96" align="center-left"/>
 </instance>
-<instance part="L2-7,5NH1" gate="G$1" x="482.6" y="-53.34" smashed="yes">
-<attribute name="NAME" x="483.87" y="-54.61" size="1.778" layer="95" align="center-left"/>
-<attribute name="VALUE" x="483.87" y="-57.15" size="1.778" layer="96" align="center-left"/>
+<instance part="L2-7,5NH1" gate="G$1" x="490.22" y="-53.34" smashed="yes">
+<attribute name="NAME" x="491.49" y="-54.61" size="1.778" layer="95" align="center-left"/>
+<attribute name="VALUE" x="491.49" y="-57.15" size="1.778" layer="96" align="center-left"/>
 </instance>
 <instance part="IC7" gate="G$1" x="355.6" y="63.5" smashed="yes">
@@
 </segment>
 <segment>
-<pinref part="R18" gate="G$1" pin="1"/>
-<pinref part="GND21" gate="1" pin="GND"/>
-<wire x1="448.282" y1="44.148" x2="448.282" y2="39.576" width="0.1524" layer="91"/>
-</segment>
-<segment>
 <pinref part="GND22" gate="1" pin="GND"/>
 <pinref part="C12" gate="G$1" pin="2"/>
@@
 <label x="693.42" y="17.78" size="1.27" layer="95" xref="yes"/>
 </segment>
+<segment>
+<pinref part="IC2" gate="G$1" pin="TEMP"/>
+<pinref part="GND21" gate="1" pin="GND"/>
+<wire x1="480.54" y1="56.34" x2="448.282" y2="56.34" width="0.1524" layer="91"/>
+<wire x1="448.282" y1="56.34" x2="448.282" y2="39.576" width="0.1524" layer="91"/>
+</segment>
 </net>
 <net name="N$9" class="0">
@@
 <pinref part="JP2" gate="A" pin="27"/>
 </segment>
+<segment>
+<pinref part="U6" gate="G$1" pin="SCS/CMD"/>
+<wire x1="596.9" y1="-25.4" x2="594.36" y2="-25.4" width="0.1524" layer="91"/>
+<label x="594.36" y="-25.4" size="1.27" layer="95" rot="R180" xref="yes"/>
+</segment>
 </net>
 <net name="N$16" class="0">
@@
 <pinref part="U3" gate="G$1" pin="RXD"/>
 </segment>
-<segment>
-<pinref part="U6" gate="G$1" pin="IO17"/>
-<wire x1="637.54" y1="-17.78" x2="640.08" y2="-17.78" width="0.1524" layer="91"/>
-<label x="640.08" y="-17.78" size="1.27" layer="95" xref="yes"/>
-</segment>
 </net>
 <net name="UART_RX_BUS" class="0">
@@
 <label x="520.7" y="142.24" size="1.778" layer="95"/>
 <pinref part="U3" gate="G$1" pin="TXD"/>
-</segment>
-<segment>
-<pinref part="U6" gate="G$1" pin="IO16"/>
-<wire x1="637.54" y1="-15.24" x2="640.08" y2="-15.24" width="0.1524" layer="91"/>
-<label x="640.08" y="-15.24" size="1.27" layer="95" xref="yes"/>
 </segment>
 </net>
@@
 <pinref part="STD1" gate="G$1" pin="C"/>
 <wire x1="523.72" y1="66.5" x2="523.72" y2="69.04" width="0.1524" layer="91"/>
-</segment>
-</net>
-<net name="N$37" class="0">
-<segment>
-<pinref part="R17" gate="G$1" pin="1"/>
-<pinref part="R18" gate="G$1" pin="2"/>
-<pinref part="IC2" gate="G$1" pin="TEMP"/>
-<wire x1="448.282" y1="62.182" x2="448.282" y2="56.34" width="0.1524" layer="91"/>
-<wire x1="448.282" y1="54.308" x2="448.282" y2="56.34" width="0.1524" layer="91"/>
-<wire x1="448.282" y1="56.34" x2="480.54" y2="56.34" width="0.1524" layer="91"/>
-<junction x="448.282" y="56.34"/>
 </segment>
 </net>
@@
 <wire x1="430.5" y1="64.6" x2="436.88" y2="64.6" width="0.1524" layer="91"/>
 <wire x1="436.88" y1="64.6" x2="436.88" y2="76.2" width="0.1524" layer="91"/>
-<wire x1="436.88" y1="76.2" x2="448.282" y2="76.2" width="0.1524" layer="91"/>
+<wire x1="436.88" y1="76.2" x2="448.31" y2="76.2" width="0.1524" layer="91"/>
 <wire x1="448.31" y1="76.2" x2="462.28" y2="76.2" width="0.1524" layer="91"/>
 <wire x1="462.28" y1="76.2" x2="472.44" y2="76.2" width="0.1524" layer="91"/>
@@
 <wire x1="462.28" y1="48.72" x2="462.28" y2="76.2" width="0.1524" layer="91"/>
 <junction x="462.28" y="76.2"/>
-<pinref part="R17" gate="G$1" pin="2"/>
-<wire x1="448.282" y1="72.342" x2="448.282" y2="76.2" width="0.1524" layer="91"/>
-<wire x1="448.282" y1="76.2" x2="448.31" y2="76.2" width="0.1524" layer="91"/>
 <junction x="448.31" y="76.2"/>
 <junction x="508.508" y="78.74"/>
@@
 <pinref part="L2-7,5NH1" gate="G$1" pin="2"/>
 <pinref part="C18" gate="G$1" pin="1"/>
-<wire x1="502.92" y1="-53.34" x2="505.46" y2="-53.34" width="0.1524" layer="91"/>
-</segment>
-</net>
+<wire x1="497.84" y1="-53.34" x2="505.46" y2="-53.34" width="0.1524" layer="91"/>
+</segment>
+</net>

Commit message: Add files via upload
Parts:
- 3V3, TX1: value Red -> (none)
- C12: value 10uf -> 10uF
- C2: value 0.1u -> 0.1uF
- C20: value 1onF -> 10nF
- R1: value 220R -> 220
- R14: value 1.5K -> 1.5k
- R2: value 120R -> 120
- R3, R4: value 1K -> 1k
- R5: value 100K -> 100k
- R6: value 6.8K -> 6.8k
- R7: value 26.1K -> 26.1k
- R8: value 10K -> 10k
- RX1: value Green -> (none)
Other:
- note added: "EESC - USP"
- note added: "Julho 2020"
- note added: "Leonardo Baptistella, Gabriel Garofa e Felipe Casseb"
